File: kicad/intensity_pi.kicad_pcb (KiCad board)
At the start: 4 copper layers, 64.4 x 171.2 mm, 127 parts, among them J1 Input A, J2 Input B / Setpoint, J3 Monitor, J4 Output, J7 select 1, J8 Screw_Terminal_01x03, Q1 2N7002E, Q2 2N7002E, SW1 SW_SPDT, SW2 SW_SPDT, SW3 SW_SPDT, SW5 EG6100-ND, U1 LM4040DBZ-5, U10 OPA189, U11 PC817, U12 OPA189, U13 BUF634A, U14 TMUX6123, U17 TMUX6123, U18 OPA189, U19 L7815, U2 LM4040DBZ-5, U20 OPA189, U21 OPA189, U22 4x Comparator, U23 L7915, U3 INA849, U4 INA849, U5 OPA189, U7 OPA189, U8 BUF634A, U9 LM317_TO-252

Commit message: different way to route design
Parts:
- added R41: 1k, Resistor_SMD:R_0805_2012Metric, F.Cu at (238.0, 71.5)
- moved D3 139.7 mm to (154.5, 96.0)
- moved C25 131.4 mm to (142.2, 110.0)
- moved C26 131.4 mm to (147.9, 118.9)
- moved C31 131.4 mm to (138.4, 120.7)
- moved C36 131.4 mm to (144.2, 109.5)
- moved C37 131.4 mm to (154.6, 113.1)
- moved Q1 131.4 mm to (155.7, 109.2)
- moved Q2 131.4 mm to (149.4, 102.6)
- moved R11 131.4 mm to (138.5, 117.2)
- moved R28 131.4 mm to (146.6, 100.8)
- moved R29 131.4 mm to (143.3, 112.9)
- moved R30 131.4 mm to (147.7, 106.1)
- moved R31 131.4 mm to (143.3, 114.8)
- moved R32 131.4 mm to (153.2, 106.1)
- moved R38 131.4 mm to (153.2, 104.2)
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Connections:
- U7 pad 3: Error_signal -> Net-(U7-+)
Routing:
- net Net-(R44-Pad1): track 123.0 -> 12.5 mm, vias 1 -> 0
- net Net-(SW2-A): track 148.0 -> 43.2 mm
- net Net-(D1-A): track 152.3 -> 51.0 mm, vias 1 -> 2
- net Net-(U20-+): track 97.6 -> 0.65 mm, vias 2 -> 1
- net Net-(R16-Pad2): track 84.2 -> 7.63 mm, vias 2 -> 0
- net Net-(U7-+): track 0.00 -> 66.7 mm, vias 0 -> 2
- net Error_signal: track 154.7 -> 94.9 mm, vias 3 -> 2
- net Net-(SW1-A): track 60.5 -> 6.38 mm
- net Net-(R12-Pad2): track 52.0 -> 25.5 mm
- net Net-(R13-Pad1): track 7.67 -> 33.3 mm
- net Net-(U14C-SEL1): track 36.8 -> 11.9 mm, vias 1 -> 0
- net Net-(D3-K1): track 23.9 -> 0.00 mm
- net Net-(D3-K2): track 21.5 -> 0.00 mm
- net Vlim+: track 32.1 -> 14.9 mm
- net Net-(D3-A): track 23.6 -> 8.82 mm
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